Commit message: Added uv and cycle test code

File: urdf_files/urdf/quadruped.urdf (robot description, URDF)
Before this commit: robot urdf_assembly, 13 links, 12 joints
Links:
- added link FL_foot, mass 0.01; collision sphere radius=0.015; visual sphere radius=0.015
- added link FR_foot, mass 0.01; collision sphere radius=0.015; visual sphere radius=0.015
- added link RL_foot, mass 0.01; collision sphere radius=0.015; visual sphere radius=0.015
- added link RR_foot, mass 0.01; collision sphere radius=0.015; visual sphere radius=0.015
- link base_link: mass 136.10446748631816 -> 5.037930; geometry collision mesh filename=./meshes/base_link.stl scale=0.001 0.001 0.001; visual mesh filename=./meshes/base_link.stl scale=0.001 0.001 0.001
- link calf_link1_1: geometry collision mesh filename=./meshes/calf_link1_1.stl scale=0.001 0.001 0.001; visual mesh filename=./meshes/calf_link1_1.stl scale=0.001 0.001 0.001
- link calf_link2_1: geometry collision mesh filename=./meshes/calf_link2_1.stl scale=0.001 0.001 0.001; visual mesh filename=./meshes/calf_link2_1.stl scale=0.001 0.001 0.001
- link calf_link3_1: geometry collision mesh filename=./meshes/calf_link3_1.stl scale=0.001 0.001 0.001; visual mesh filename=./meshes/calf_link3_1.stl scale=0.001 0.001 0.001
- link calf_link4_1: geometry collision mesh filename=./meshes/calf_link4_1.stl scale=0.001 0.001 0.001; visual mesh filename=./meshes/calf_link4_1.stl scale=0.001 0.001 0.001
- link hip_abduction2_1: geometry collision mesh filename=./meshes/hip_abduction2_1.stl scale=0.001 0.001 0.001; visual mesh filename=./meshes/hip_abduction2_1.stl scale=0.001 0.001 0.001
- link hip_abduction3_1: geometry collision mesh filename=./meshes/hip_abduction3_1.stl scale=0.001 0.001 0.001; visual mesh filename=./meshes/hip_abduction3_1.stl scale=0.001 0.001 0.001
- link hip_abduction4_1: geometry collision mesh filename=./meshes/hip_abduction4_1.stl scale=0.001 0.001 0.001; visual mesh filename=./meshes/hip_abduction4_1.stl scale=0.001 0.001 0.001
- link hip_abduction_1: geometry collision mesh filename=./meshes/hip_abduction_1.stl scale=0.001 0.001 0.001; visual mesh filename=./meshes/hip_abduction_1.stl scale=0.001 0.001 0.001
- link thigh_link1_1: geometry collision mesh filename=./meshes/thigh_link1_1.stl scale=0.001 0.001 0.001; visual mesh filename=./meshes/thigh_link1_1.stl scale=0.001 0.001 0.001
- link thigh_link2_1: geometry collision mesh filename=./meshes/thigh_link2_1.stl scale=0.001 0.001 0.001; visual mesh filename=./meshes/thigh_link2_1.stl scale=0.001 0.001 0.001
- link thigh_link3_1: geometry collision mesh filename=./meshes/thigh_link3_1.stl scale=0.001 0.001 0.001; visual mesh filename=./meshes/thigh_link3_1.stl scale=0.001 0.001 0.001
- link thigh_link4_1: geometry collision mesh filename=./meshes/thigh_link4_1.stl scale=0.001 0.001 0.001; visual mesh filename=./meshes/thigh_link4_1.stl scale=0.001 0.001 0.001
Joints:
- removed joint Revolute_1
- removed joint Revolute_10
- removed joint Revolute_11
- removed joint Revolute_12
- removed joint Revolute_2
- removed joint Revolute_3
- removed joint Revolute_4
- removed joint Revolute_5
- removed joint Revolute_6
- removed joint Revolute_7
- removed joint Revolute_8
- removed joint Revolute_9
- added joint FL_calf_joint: type continuous, parent thigh_link4_1, child calf_link4_1, origin xyz=-0.0541 -0.15 -0.259808 rpy=0 0 0, axis 1.0 -0.0 0.0, limit lower=-1.5708 upper=1.5708
- added joint FL_foot_joint: type continuous, parent calf_link4_1, child FL_foot, origin xyz=-0.01 0.145 -0.24 rpy=0 0 0, limit lower=0 upper=0
- added joint FL_hip_joint: type continuous, parent base_link, child hip_abduction2_1, origin xyz=-0.11 0.053 4e-06 rpy=0 0 0, axis 0.0 1.0 0.0, limit lower=-1.5708 upper=1.5708
- added joint FL_thigh_joint: type continuous, parent hip_abduction2_1, child thigh_link4_1, origin xyz=-0.0274 0.058 0.0 rpy=0 0 0, axis -1.0 0.0 -0.0, limit lower=-1.5708 upper=1.5708
- added joint FR_calf_joint: type continuous, parent thigh_link2_1, child calf_link2_1, origin xyz=0.0765 -0.15 -0.259808 rpy=0 0 0, axis -1.0 -0.0 -0.0, limit lower=-1.5708 upper=1.5708
- added joint FR_foot_joint: type continuous, parent calf_link2_1, child FR_foot, origin xyz=-0.01 0.145 -0.24 rpy=0 0 0, limit lower=0 upper=0
- added joint FR_hip_joint: type continuous, parent base_link, child hip_abduction_1, origin xyz=0.11 0.053 4e-06 rpy=0 0 0, axis 0.0 1.0 0.0, limit lower=-1.5708 upper=1.5708
- added joint FR_thigh_joint: type continuous, parent hip_abduction_1, child thigh_link2_1, origin xyz=0.0274 0.058 0.0 rpy=0 0 0, axis 1.0 -0.0 0.0, limit lower=-1.5708 upper=1.5708
- added joint RL_calf_joint: type continuous, parent thigh_link3_1, child calf_link3_1, origin xyz=-0.0541 -0.15 -0.259808 rpy=0 0 0, axis 1.0 -0.0 0.0, limit lower=-1.5708 upper=1.5708
- added joint RL_foot_joint: type continuous, parent calf_link3_1, child RL_foot, origin xyz=-0.01 0.145 -0.24 rpy=0 0 0, limit lower=0 upper=0
- added joint RL_hip_joint: type continuous, parent base_link, child hip_abduction3_1, origin xyz=-0.11 -0.553 4e-06 rpy=0 0 0, axis -0.0 -1.0 -0.0, limit lower=-1.5708 upper=1.5708
- added joint RL_thigh_joint: type continuous, parent hip_abduction3_1, child thigh_link3_1, origin xyz=-0.0274 -0.058 0.0 rpy=0 0 0, axis -1.0 0.0 -0.0, limit lower=-1.5708 upper=1.5708
- added joint RR_calf_joint: type continuous, parent thigh_link1_1, child calf_link1_1, origin xyz=0.0541 -0.15 -0.259808 rpy=0 0 0, axis 1.0 0.0 -0.0, limit lower=-1.5708 upper=1.5708
- added joint RR_foot_joint: type continuous, parent calf_link1_1, child RR_foot, origin xyz=0.01 0.145 -0.24 rpy=0 0 0, limit lower=0 upper=0
- added joint RR_hip_joint: type continuous, parent base_link, child hip_abduction4_1, origin xyz=0.11 -0.553 4e-06 rpy=0 0 0, axis -0.0 -1.0 -0.0, limit lower=-1.5708 upper=1.5708
- added joint RR_thigh_joint: type continuous, parent hip_abduction4_1, child thigh_link1_1, origin xyz=0.0274 -0.058 0.0 rpy=0 0 0, axis 1.0 -0.0 0.0, limit lower=-1.5708 upper=1.5708
