Commit message: checkpoint

File: src/ga_quadruped/assets/param/param.urdf (robot description, URDF)
Before this commit: robot urdf_assembly_v3, 14 links, 13 joints
Links:
- added link world
Joints:
- added joint world_to_base_rotX180: type fixed, parent world, child trunk, origin xyz=0 0 0 rpy=0 0 3.141592653589793
