Commit message: Jump Env Checkpoint

File: assets/param/param.urdf (robot description, URDF)
Before this commit: robot urdf_assembly_v3, 15 links, 14 joints
Joints:
- joint FL_hip_joint: limit lower=-0.785 upper=0.785 -> lower=0 upper=6.28
- joint RL_hip_joint: limit lower=-0.785 upper=0.785 -> lower=0 upper=6.28
- joint RR_hip_joint: limit lower=-0.785 upper=0.785 -> lower=0 upper=6.28

Commit message: Ramp policy

File: assets/param/param.urdf (robot description, URDF)
Before this commit: robot urdf_assembly_v3, 15 links, 14 joints
Joints:
- joint FL_hip_joint: limit lower=0 upper=6.28 -> lower=-3.14 upper=3.14
- joint FR_hip_joint: limit lower=-0.785 upper=0.785 -> lower=-3.14 upper=3.14
- joint RL_hip_joint: limit lower=0 upper=6.28 -> lower=-3.14 upper=3.14
- joint RR_hip_joint: limit lower=0 upper=6.28 -> lower=-3.14 upper=3.14
